Commit message: Wheel collision was modified

File: urdf/ros2_control.urdf.xacro (robot description, xacro)
@@ -3,4 +3,10 @@
   <xacro:macro name="ros2_control">
       <gazebo>
+        <plugin
+          filename="gz-sim-odometry-publisher-system"
+          name="gz::sim::systems::OdometryPublisher">
+          <odom_frame>odom</odom_frame>
+          <robot_base_frame>base_footprint</robot_base_frame>
+        </plugin>
         <plugin filename="libgz_ros2_control-system.so" name="gz_ros2_control::GazeboSimROS2ControlPlugin">
           <ros>

File: urdf/wheels/rubber_wheel/rubber_wheel.urdf.xacro (robot description, xacro)
@@ -45,8 +45,10 @@
           </xacro:unless>
           <xacro:if value="${reflect}">
-            <origin xyz="0 0 0" rpy="${M_PI} 0 0" />
+            <origin xyz="0 0 0" rpy="${M_PI/2} 0 0" />
+            <!-- <origin xyz="0 0 0" rpy="${M_PI} 0 0" /> -->
           </xacro:if>
           <geometry>
-						<mesh filename="package://${mesh_file}.stl" />
+            <cylinder length="${rubber_wheel_width}" radius="${rubber_wheel_radius}" />
+						<!-- <mesh filename="package://${mesh_file}.stl" /> -->
         </geometry>
       </collision>
