Commit message: Support for Gazebo Harmonic

File: robots/summit_xl_std.urdf.xacro (robot description, xacro)
@@ -1,103 +1,85 @@
 <?xml version="1.0"?>
 <robot name="summit_xl" xmlns:xacro="http://wiki.ros.org/xacro">
-	<!-- ***************** -->
-	<!-- Imported elements -->
-	<!-- ***************** -->
-	<!-- First we import all posible elements defined in the urdf.xacro files. All these elements are defined as macro:xacros -->
-	<!-- Import summit XL base elements -->
-	<xacro:include filename="$(find robot_description)/urdf/bases/summit_xl_base.urdf.xacro" />
-	<!-- Import summit XL wheels -->
-	<xacro:include filename="$(find robot_description)/urdf/wheels/rubber_wheel/rubber_wheel.urdf.xacro" />
-  <xacro:include filename="$(find robot_description)/urdf/wheels/omni_wheel/omni_wheel.urdf.xacro" />
-	<!-- Import all available sensors -->
-	<xacro:include filename="$(find robotnik_sensors)/urdf/all_sensors.urdf.xacro" />
-	<!-- Import antenna -->
-	<xacro:include filename="$(find robot_description)/urdf/structures/sensor_support/structure_teltonika.urdf.xacro" />
-	<xacro:property name="PI" value="3.1415926535897931"/>
-	<!-- Wheel parameters -->
-	<xacro:property name="wheel_offset_x" value="0.229" />    <!-- x,y,z in translation from base_link to the center of the wheel -->
-	<xacro:property name="wheel_offset_y" value="0.235" />
-	<xacro:property name="wheel_offset_z" value="0.0" />
-	<!-- Flag to select the high or low quality model -->
-	<xacro:property name="hq" value="true" />
-	<xacro:arg name="prefix" default="summit_xl_"/>
-	<xacro:arg name="ros_planar_move_plugin" default="false"/>
-    <xacro:arg name="ros_planar_move_plugin_force_based" default="false"/>
-	<xacro:arg name="kinematics" default="skid"/>
-	<xacro:arg name="gpu" default="false"/>
-	<xacro:arg name="gps_latitude" default="0"/>
-	<xacro:arg name="gps_longitude" default="0"/>
-    <xacro:macro name="summit_xl" params="prefix publish_bf hq kinematics">
-	  <xacro:property name="mesh_file_left" value="robot_description/meshes/wheels/rubber_wheel/rubber_wheel_left" />
-	  <xacro:property name="mesh_file_right" value="robot_description/meshes/wheels/rubber_wheel/rubber_wheel_right" />
-		<!-- *************** -->
-		<!-- Robots Elements -->
-		<!-- *************** -->
-		<!-- Here we create the robot elements using the xacro:macros imported at the beggining of this file -->
-		<!-- Summit XL base -->
-		<xacro:summit_xl_base prefix="$(arg prefix)" publish_bf="true" hq="${hq}" />
-    <xacro:if value="${kinematics == 'skid' or kinematics == 'skid_4w'}">
-  		<xacro:rubber_wheel prefix="$(arg prefix)front_right" parent="$(arg prefix)base_link" reflect="false" hq="${hq}" mesh_file="${mesh_file_right}">
-  			<origin xyz="${wheel_offset_x} -${wheel_offset_y} ${wheel_offset_z}" rpy="0 0 0"/>
-  		</xacro:rubber_wheel>
-  		<xacro:rubber_wheel prefix="$(arg prefix)front_left" parent="$(arg prefix)base_link" reflect="false" hq="${hq}" mesh_file="${mesh_file_left}">
-  			<origin xyz="${wheel_offset_x} ${wheel_offset_y} ${wheel_offset_z}" rpy="0 0 0"/>
-  		</xacro:rubber_wheel>
-  		<xacro:rubber_wheel prefix="$(arg prefix)back_left" parent="$(arg prefix)base_link" reflect="false" hq="${hq}" mesh_file="${mesh_file_left}">
-  			<origin xyz="-${wheel_offset_x} ${wheel_offset_y} ${wheel_offset_z}" rpy="0 0 0"/>
-  		</xacro:rubber_wheel>
-  		<xacro:rubber_wheel prefix="$(arg prefix)back_right" parent="$(arg prefix)base_link" reflect="false" hq="${hq}" mesh_file="${mesh_file_right}">
-  			<origin xyz="-${wheel_offset_x} -${wheel_offset_y} ${wheel_offset_z}" rpy="0 0 0"/>
-  		</xacro:rubber_wheel>
-    </xacro:if>
-    <xacro:if value="${kinematics == 'omni' or kinematics == 'omni_4w'}">
-  		<xacro:omni_wheel prefix="$(arg prefix)front_right" parent="$(arg prefix)base_link" reflect="false" hq="${hq}">
-  			<origin xyz="${wheel_offset_x} -${wheel_offset_y} ${wheel_offset_z}" rpy="0 0 0"/>
-  		</xacro:omni_wheel>
-  		<xacro:omni_wheel prefix="$(arg prefix)front_left" parent="$(arg prefix)base_link" reflect="true" hq="${hq}">
-  			<origin xyz="${wheel_offset_x} ${wheel_offset_y} ${wheel_offset_z}" rpy="0 0 0"/>
-  		</xacro:omni_wheel>
-  		<xacro:omni_wheel prefix="$(arg prefix)back_left" parent="$(arg prefix)base_link" reflect="true" hq="${hq}">
-  			<origin xyz="-${wheel_offset_x} ${wheel_offset_y} ${wheel_offset_z}" rpy="0 0 0"/>
-  		</xacro:omni_wheel>
-  		<xacro:omni_wheel prefix="$(arg prefix)back_right" parent="$(arg prefix)base_link" reflect="false" hq="${hq}">
-  			<origin xyz="-${wheel_offset_x} -${wheel_offset_y} ${wheel_offset_z}" rpy="0 0 0"/>
-  		</xacro:omni_wheel>
-    </xacro:if>
-        <!-- IMU -->
-		<xacro:sensor_imu prefix="$(arg prefix)imu" parent="$(arg prefix)base_link" topic="imu/data_raw">
-			<origin xyz="0.0385 0.132 0.158" rpy="0 0 0"/>
-		</xacro:sensor_imu>
-		<!-- 3d laser -->
-		<xacro:sensor_rs_helios_16p prefix="$(arg prefix)top_3d_laser" parent="$(arg prefix)base_link" gpu="$(arg gpu)">
-			<origin xyz="-0.11808 0.0 0.38509" rpy="0 0 0"/>
-		</xacro:sensor_rs_helios_16p>
-		<!-- ptz camera -->
-		<!--xacro:sensor_axis prefix="$(arg prefix)front_ptz_camera" parent="$(arg prefix)base_link">
-			<origin xyz="0.19 0 0.26" rpy="0 ${15*PI/180} 0"/>
-		</xacro:sensor_axis-->
-	  <!-- RGBD -->
-	  <xacro:sensor_orbbec_astra prefix="$(arg prefix)front_rgbd_camera" parent="$(arg prefix)base_link" prefix_topic="front_rgbd_camera">
-			<origin xyz="0.324 0.012 0.172" rpy="0 0 0"/>
-		</xacro:sensor_orbbec_astra>
-	  <!-- GPS -->
-	  <xacro:sensor_gps_with_mast prefix="$(arg prefix)gps" parent="$(arg prefix)base_link" gps_latitude="$(arg gps_latitude)" gps_longitude="$(arg gps_longitude)" update_rate="5">
-			<origin xyz="-0.22528 0.095 0.275" rpy="0 0 0"/>
-		</xacro:sensor_gps_with_mast>
-	  <!--Antenna-->
-	  <xacro:structure_mastil_teltonika prefix="$(arg prefix)antenna" parent="$(arg prefix)base_link">
-			<origin xyz="-0.22528 -0.095 0.23325" rpy="0 0 0"/>
-		</xacro:structure_mastil_teltonika>
-	  <!-- Gazebo ros control pluggins -->
-      <xacro:ros_control/>
-	  <xacro:if value="$(arg ros_planar_move_plugin)">
-		<xacro:if value="${kinematics == 'omni' or kinematics == 'omni_4w'}">
-			<xacro:omni_steering prefix="$(arg prefix)" publish_tf="true" force_based="$(arg ros_planar_move_plugin_force_based)"/>
-		</xacro:if>
-		<xacro:if value="${kinematics == 'skid' or kinematics == 'skid_4w'}">
-			<xacro:skid_steering prefix="$(arg prefix)" publish_tf="true" force_based="$(arg ros_planar_move_plugin_force_based)"/>
-		</xacro:if>
-	  </xacro:if>
-   </xacro:macro>
-   <xacro:summit_xl prefix="$(arg prefix)" publish_bf="true" hq="true" kinematics="$(arg kinematics)"/>
+  <!-- ***************** -->
+  <!-- Imported elements -->
+  <!-- ***************** -->
+  <!-- Import RB1 base elements (base + wheels) -->
+  <xacro:include filename="$(find robot_description)/urdf/bases/summit_xl_base.urdf.xacro"/>
+  <xacro:include filename="$(find robot_description)/urdf/wheels/rubber_wheel/rubber_wheel.urdf.xacro"/>
+  <xacro:include filename="$(find robot_description)/urdf/wheels/omni_wheel/omni_wheel.urdf.xacro"/>
+  <xacro:include filename="$(find robot_description)/urdf/structures/sensor_support/structure_gps.urdf.xacro"/>
+  <!-- Import all available sensors -->
+  <xacro:include filename="$(find robotnik_sensors)/urdf/all_sensors.urdf.xacro"/>
+  <!-- ***************** -->
+  <!-- Global parameters -->
+  <!-- ***************** -->
+  <xacro:property name="PI" value="3.1415926535897931"/>
+  <!-- Wheel parameters -->
+  <!-- x,y,z in translation from base_link to the center of the wheel -->
+  <xacro:property name="wheel_offset_x" value="0.229"/>
+  <xacro:property name="wheel_offset_y" value="0.235"/>
+  <xacro:property name="wheel_offset_z" value="0.0"/>
+  <!-- Flag to select the high or low quality model -->
+  <xacro:property name="hq" value="true"/>
+  <xacro:arg name="robot_id" default="summit_xl"/>
+  <xacro:arg name="prefix" default=""/>
+  <xacro:arg name="robot_ns" default=""/>
+  <xacro:arg name="omni_wheels" default="false"/>
+  <xacro:arg name="use_sim_time" default="true"/>
+  <!-- *************** -->
+  <!-- Robots Elements -->
+  <!-- *************** -->
+  <!-- Summit XL -->
+  <xacro:summit_xl_base prefix="$(arg prefix)" publish_bf="true" hq="${hq}"/>
+  <!--xacro:gazebo_colors /-->
+  <!-- WHEELS -->
+  <xacro:unless value="$(arg omni_wheels)">
+    <xacro:rubber_wheel prefix="front_right_" parent="$(arg prefix)base_link" reflect="true" hq="${hq}">
+      <origin xyz="${wheel_offset_x} -${wheel_offset_y} ${wheel_offset_z}" rpy="0 0 ${PI}"/>
+    </xacro:rubber_wheel>
+    <xacro:rubber_wheel prefix="front_left_" parent="$(arg prefix)base_link" reflect="true" hq="${hq}">
+      <origin xyz="${wheel_offset_x} ${wheel_offset_y} ${wheel_offset_z}" rpy="0 0 0"/>
+    </xacro:rubber_wheel>
+    <xacro:rubber_wheel prefix="rear_left_" parent="$(arg prefix)base_link" reflect="true" hq="${hq}">
+      <origin xyz="-${wheel_offset_x} ${wheel_offset_y} ${wheel_offset_z}" rpy="0 0 0"/>
+    </xacro:rubber_wheel>
+    <xacro:rubber_wheel prefix="rear_right_" parent="$(arg prefix)base_link" reflect="true" hq="${hq}">
+      <origin xyz="-${wheel_offset_x} -${wheel_offset_y} ${wheel_offset_z}" rpy="0 0 ${PI}"/>
+    </xacro:rubber_wheel>
+  </xacro:unless>
+  <xacro:if value="$(arg omni_wheels)">
+    <xacro:omni_wheel prefix="front_right_" parent="$(arg prefix)base_link" reflect="true" hq="${hq}">
+      <origin xyz="${wheel_offset_x} -${wheel_offset_y} ${wheel_offset_z}" rpy="0 0 ${PI}"/>
+    </xacro:omni_wheel>
+    <xacro:omni_wheel prefix="front_left_" parent="$(arg prefix)base_link" reflect="true" hq="${hq}">
+      <origin xyz="${wheel_offset_x} ${wheel_offset_y} ${wheel_offset_z}" rpy="0 0 0"/>
+    </xacro:omni_wheel>
+    <xacro:omni_wheel prefix="back_left_" parent="$(arg prefix)base_link" reflect="true" hq="${hq}">
+      <origin xyz="-${wheel_offset_x} ${wheel_offset_y} ${wheel_offset_z}" rpy="0 0 0"/>
+    </xacro:omni_wheel>
+    <xacro:omni_wheel prefix="back_right_" parent="$(arg prefix)base_link" reflect="true" hq="${hq}">
+      <origin xyz="-${wheel_offset_x} -${wheel_offset_y} ${wheel_offset_z}" rpy="0 0 ${PI}"/>
+    </xacro:omni_wheel>
+  </xacro:if>
+  <!-- SENSORS -->
+  <xacro:sensor_robosense_helios node_namespace="$(arg robot_ns)" frame_prefix="$(arg prefix)front_laser_" parent="$(arg prefix)base_link" simulation="true" gpu="true">
+      <origin xyz="-0.11808 0.0 0.38509" rpy="0 0 0"/>
+  </xacro:sensor_robosense_helios>
+  <xacro:sensor_stereolabs_zed2 node_namespace="$(arg robot_ns)" frame_prefix="$(arg prefix)front_camera_" parent="$(arg prefix)base_link" simulation="true">
+      <origin xyz="0.324 0.012 0.172" rpy="0 0 0"/>
+  </xacro:sensor_stereolabs_zed2>
+  <xacro:structure_mastil_gps prefix="$(arg prefix)gps_" parent="$(arg prefix)base_link">
+    <origin xyz="-0.24 0.095 0.25" rpy="0 0 0"/>
+  </xacro:structure_mastil_gps>
+  <xacro:sensor_gps  node_namespace="$(arg robot_ns)" frame_prefix="$(arg prefix)gps_" parent="$(arg prefix)base_link" simulation="true">
+    <origin xyz="-0.24 0.095 0.625" rpy="0 0 0"/>
+  </xacro:sensor_gps>
+  <xacro:sensor_imu ns="$(arg robot_ns)" prefix="$(arg prefix)imu" parent="$(arg prefix)base_link">
+    <origin xyz="0.0 0.0 0.0" rpy="0 0 0"/>
+  </xacro:sensor_imu>
+  <!-- Gazebo ros control plugins -->
+  <xacro:arg name="config_controllers" default="$(find robot_description)/config/summit_controllers.yaml"/>
+  <xacro:arg name="update_rate" default="100"/>
+  <xacro:include filename="$(find robot_description)/urdf/ros2_control.urdf.xacro"/>
+  <xacro:ros2_control/>
 </robot>

File: robots/summit_xls_std.urdf.xacro (robot description, xacro)
@@ -1,96 +1,87 @@
 <?xml version="1.0"?>
 <robot name="summit_xl" xmlns:xacro="http://wiki.ros.org/xacro">
-	<!-- ***************** -->
-	<!-- Imported elements -->
-	<!-- ***************** -->
-	<!-- First we import all posible elements defined in the urdf.xacro files. All these elements are defined as macro:xacros -->
-	<!-- Import summit XL base elements -->
-	<xacro:include filename="$(find robot_description)/urdf/bases/summit_xl_steel_base.urdf.xacro" />
-	<!-- Import summit XL wheels -->
-	<xacro:include filename="$(find robot_description)/urdf/wheels/omni_wheel/omni_wheel.urdf.xacro" />
-	<xacro:include filename="$(find robot_description)/urdf/wheels/rubber_wheel/rubber_wheel.urdf.xacro" />
-	<xacro:include filename="$(find robot_description)/urdf/structures/rbkairos_chassis/structure_hokuyo.urdf.xacro" />
-	<!-- Import all available sensors -->
-	<xacro:include filename="$(find robotnik_sensors)/urdf/all_sensors.urdf.xacro" />
-	<xacro:property name="PI" value="3.1415926535897931"/>
-	<!-- Wheel parameters -->
-	<!-- Wheel parameters -->
-	<xacro:property name="wheel_offset_x" value="0.2225" />    <!-- x,y,z in translation from base_link to the center of the wheel -->
-	<xacro:property name="wheel_offset_y" value="0.2045" />
-	<xacro:property name="wheel_offset_z" value="0.0" />
-	<xacro:property name="front_laser_offset_x" value="0.2865"/>
-	<xacro:property name="front_laser_offset_y" value="-0.20894"/>
-	<xacro:property name="front_laser_offset_z" value="0.2973"/>
-	<xacro:property name="rear_laser_offset_x" value="-0.2865"/>
-	<xacro:property name="rear_laser_offset_y" value="0.20894"/>
-	<xacro:property name="rear_laser_offset_z" value="0.2973"/>
-	<xacro:property name="front_ptz_camera_offset_x" value="0.308"/>
-	<xacro:property name="front_ptz_camera_offset_y" value="0.141"/>
-	<xacro:property name="front_ptz_camera_offset_z" value="0.195"/>
-	<xacro:property name="rear_ptz_camera_offset_x" value="-0.308"/>
-	<xacro:property name="rear_ptz_camera_offset_y" value="-0.141"/>
-	<xacro:property name="rear_ptz_camera_offset_z" value="0.195"/>
-	<xacro:property name="imu_offset_x" value="0.127"/>
-	<xacro:property name="imu_offset_y" value="-0.129"/>
-	<xacro:property name="imu_offset_z" value="0.212"/>
-	<xacro:property name="front_rgbd_camera_offset_x" value="0.35850"/>
-	<xacro:property name="front_rgbd_camera_offset_y" value="0.0"/>
-	<xacro:property name="front_rgbd_camera_offset_z" value="0.25062"/>
-	<xacro:property name="gps_offset_x" value="-0.365"/>
-	<xacro:property name="gps_offset_y" value="-0.167"/>
-	<xacro:property name="gps_offset_z" value="0.302"/>
-	<!-- Flag to select the high or low quality model -->
-	<xacro:property name="hq" value="true" />
-	<xacro:arg name="prefix" default="summit_xl_"/>
-	<xacro:arg name="ros_planar_move_plugin" default="false"/>
-	<xacro:arg name="ros_planar_move_plugin_force_based" default="false"/>
-	<xacro:arg name="gpu" default="false"/>
-    <xacro:macro name="summit_xl" params="prefix publish_bf hq">
-		<!-- *************** -->
-		<!-- Robots Elements -->
-		<!-- *************** -->
-		<!-- Here we create the robot elements using the xacro:macros imported at the beggining of this file -->
-		<!-- Summit XL base -->
-		<xacro:summit_xl_steel_base prefix="$(arg prefix)" publish_bf="true" hq="${hq}" />
-		<xacro:omni_wheel prefix="$(arg prefix)front_right" parent="$(arg prefix)base_link" reflect="false" hq="${hq}">
-			<origin xyz="${wheel_offset_x} -${wheel_offset_y} ${wheel_offset_z}" rpy="0 0 0"/>
-		</xacro:omni_wheel>
-		<xacro:omni_wheel prefix="$(arg prefix)front_left" parent="$(arg prefix)base_link" reflect="true" hq="${hq}">
-			<origin xyz="${wheel_offset_x} ${wheel_offset_y} ${wheel_offset_z}" rpy="0 0 0"/>
-		</xacro:omni_wheel>
-		<xacro:omni_wheel prefix="$(arg prefix)back_left" parent="$(arg prefix)base_link" reflect="true" hq="${hq}">
-			<origin xyz="-${wheel_offset_x} ${wheel_offset_y} ${wheel_offset_z}" rpy="0 0 0"/>
-		</xacro:omni_wheel>
-		<xacro:omni_wheel prefix="$(arg prefix)back_right" parent="$(arg prefix)base_link" reflect="false" hq="${hq}">
-			<origin xyz="-${wheel_offset_x} -${wheel_offset_y} ${wheel_offset_z}" rpy="0 0 0"/>
-		</xacro:omni_wheel>
-        <!-- IMU -->
-		<xacro:sensor_imu prefix="$(arg prefix)imu" parent="$(arg prefix)base_link" topic="imu/data_raw">
-			<origin xyz="${imu_offset_x} ${imu_offset_y} ${imu_offset_z}" rpy="0 0 0"/>
-		</xacro:sensor_imu>
-		<!-- SENSORS -->
-		<xacro:sensor_sick_s300 prefix="$(arg prefix)front_laser" parent="$(arg prefix)base_link" prefix_topic="front_laser" gpu="$(arg gpu)">
-			<origin xyz="${front_laser_offset_x} ${front_laser_offset_y} ${front_laser_offset_z}" rpy="0 ${-PI} ${3/4*PI}" />
-		</xacro:sensor_sick_s300>
-		<xacro:sensor_sick_s300 prefix="$(arg prefix)rear_laser" parent="$(arg prefix)base_link" prefix_topic="rear_laser" gpu="$(arg gpu)">
-			<origin xyz="${rear_laser_offset_x} ${rear_laser_offset_y} ${rear_laser_offset_z}" rpy="0 ${-PI} ${-1/4*PI}" />
-		</xacro:sensor_sick_s300>
-		<!--xacro:sensor_axis_m5013 prefix="$(arg prefix)front_ptz_camera" parent="$(arg prefix)base_link">
-			<origin xyz="${front_ptz_camera_offset_x} ${front_ptz_camera_offset_y} ${front_ptz_camera_offset_z}" rpy="${-PI/2} 0 0"/>
-		</xacro:sensor_axis_m5013-->
-		<!--xacro:sensor_axis_m5013 prefix="$(arg prefix)rear_ptz_camera" parent="$(arg prefix)base_link">
-			<origin xyz="${rear_ptz_camera_offset_x} ${rear_ptz_camera_offset_y} ${rear_ptz_camera_offset_z}" rpy="${-PI/2} 0 ${PI}"/>
-		</xacro:sensor_axis_m5013-->
-		<xacro:sensor_orbbec_astra prefix="$(arg prefix)front_rgbd_camera" parent="$(arg prefix)base_link" prefix_topic="front_rgbd_camera">
-			<origin xyz="${front_rgbd_camera_offset_x} ${front_rgbd_camera_offset_y} ${front_rgbd_camera_offset_z}" rpy="0 0 0"/>
-		</xacro:sensor_orbbec_astra>
-		<!--xacro:sensor_gps prefix="$(arg prefix)gps" parent="$(arg prefix)base_link">
-			<origin xyz="${gps_offset_x} ${gps_offset_y} ${gps_offset_z}" rpy="0 0 0"/>
-		</xacro:sensor_gps-->
-   </xacro:macro>
-   <xacro:ros_control/>
-   <xacro:if value="$(arg ros_planar_move_plugin)">
-	   <xacro:omni_steering prefix="$(arg prefix)" publish_tf="true" force_based="$(arg ros_planar_move_plugin_force_based)"/>
-   </xacro:if>
-   <xacro:summit_xl prefix="$(arg prefix)" publish_bf="true" hq="true"/>
+  <!-- ***************** -->
+  <!-- Imported elements -->
+  <!-- ***************** -->
+  <!-- Import RB1 base elements (base + wheels) -->
+  <xacro:include filename="$(find robot_description)/urdf/bases/summit_xl_base.urdf.xacro"/>
+  <xacro:include filename="$(find robot_description)/urdf/wheels/rubber_wheel/rubber_wheel.urdf.xacro"/>
+  <xacro:include filename="$(find robot_description)/urdf/structures/sensor_support/gps_mast.urdf.xacro"/>
+  <!-- Import all available sensors -->
+  <xacro:include filename="$(find robotnik_sensors)/urdf/all_sensors.urdf.xacro"/>
+  <!-- ***************** -->
+  <!-- Global parameters -->
+  <!-- ***************** -->
+  <xacro:property name="PI" value="3.1415926535897931"/>
+  <!-- Wheel parameters -->
+  <!-- x,y,z in translation from base_link to the center of the wheel -->
+  <xacro:property name="wheel_offset_x" value="0.218"/>
+  <xacro:property name="wheel_offset_y" value="0.228"/>
+  <xacro:property name="wheel_offset_z" value="0.0"/>
+  <!-- Flag to select the high or low quality model -->
+  <xacro:property name="hq" value="true"/>
+  <xacro:arg name="robot_id" default="robot"/>
+  <xacro:arg name="prefix" default=""/>
+  <xacro:arg name="robot_ns" default=""/>
+  <xacro:arg name="omni_wheels" default="false"/>
+  <!-- *************** -->
+  <!-- Robots Elements -->
+  <!-- *************** -->
+  <!-- Summit XL -->
+  <xacro:summit_xl_base prefix="$(arg prefix)" publish_bf="true" hq="${hq}"/>
+  <!--xacro:gazebo_colors /-->
+  <!-- WHEELS -->
+  <xacro:unless value="$(arg omni_wheels)">
+    <xacro:rubber_wheel prefix="front_right_" parent="$(arg prefix)base_link" reflect="true" hq="${hq}">
+      <origin xyz="${wheel_offset_x} -${wheel_offset_y} ${wheel_offset_z}" rpy="0 0 ${PI}"/>
+      <axis xyz="1 0 0" rpy="0 0 0"/>
+    </xacro:rubber_wheel>
+    <xacro:rubber_wheel prefix="front_left_" parent="$(arg prefix)base_link" reflect="true" hq="${hq}">
+      <origin xyz="${wheel_offset_x} ${wheel_offset_y} ${wheel_offset_z}" rpy="0 0 0"/>
+      <axis xyz="1 0 0" rpy="0 0 0"/>
+    </xacro:rubber_wheel>
+    <xacro:rubber_wheel prefix="rear_left_" parent="$(arg prefix)base_link" reflect="true" hq="${hq}">
+      <origin xyz="-${wheel_offset_x} ${wheel_offset_y} ${wheel_offset_z}" rpy="0 0 0"/>
+      <axis xyz="1 0 0" rpy="0 0 0"/>
+    </xacro:rubber_wheel>
+    <xacro:rubber_wheel prefix="rear_right_" parent="$(arg prefix)base_link" reflect="true" hq="${hq}">
+      <origin xyz="-${wheel_offset_x} -${wheel_offset_y} ${wheel_offset_z}" rpy="0 0 ${PI}"/>
+      <axis xyz="1 0 0" rpy="0 0 0"/>
+    </xacro:rubber_wheel>
+  </xacro:unless>
+  <xacro:if value="$(arg omni_wheels)">
+    <xacro:omni_wheel prefix="front_right_" parent="$(arg prefix)base_link" reflect="true" hq="${hq}">
+      <origin xyz="${wheel_offset_x} -${wheel_offset_y} ${wheel_offset_z}" rpy="0 0 ${PI}"/>
+    </xacro:omni_wheel>
+    <xacro:omni_wheel prefix="front_left_" parent="$(arg prefix)base_link" reflect="true" hq="${hq}">
+      <origin xyz="${wheel_offset_x} ${wheel_offset_y} ${wheel_offset_z}" rpy="0 0 0"/>
+    </xacro:omni_wheel>
+    <xacro:omni_wheel prefix="back_left_" parent="$(arg prefix)base_link" reflect="true" hq="${hq}">
+      <origin xyz="-${wheel_offset_x} ${wheel_offset_y} ${wheel_offset_z}" rpy="0 0 0"/>
+    </xacro:omni_wheel>
+    <xacro:omni_wheel prefix="back_right_" parent="$(arg prefix)base_link" reflect="true" hq="${hq}">
+      <origin xyz="-${wheel_offset_x} -${wheel_offset_y} ${wheel_offset_z}" rpy="0 0 ${PI}"/>
+    </xacro:omni_wheel>
+  </xacro:if>
+  <!-- SENSORS -->
+  <xacro:sensor_robosense_helios node_namespace="$(arg robot_ns)" frame_prefix="$(arg prefix)front_laser_" parent="$(arg prefix)base_link" simulation="true" gpu="false">
+      <origin xyz="-0.11808 0.0 0.38509" rpy="0 0 0"/>
+  </xacro:sensor_robosense_helios>
+  <xacro:sensor_stereolabs_zed2 node_namespace="$(arg robot_ns)" frame_prefix="$(arg prefix)front_camera_" parent="$(arg prefix)base_link" simulation="true">
+      <origin xyz="0.324 0.012 0.172" rpy="0 0 0"/>
+  </xacro:sensor_stereolabs_zed2>
+  <xacro:sensor_gps_mast prefix="$(arg prefix)gps_" parent="$(arg prefix)base_link">
+    <origin xyz="-0.24 0.095 0.25" rpy="0 0 0"/>
+  </xacro:sensor_gps_mast>
+  <xacro:sensor_gps  node_namespace="$(arg robot_ns)" frame_prefix="$(arg prefix)gps_" parent="$(arg prefix)base_link" simulation="true">
+    <origin xyz="-0.24 0.095 0.625" rpy="0 0 0"/>
+  </xacro:sensor_gps>
+  <xacro:sensor_imu ns="$(arg robot_ns)" prefix="$(arg prefix)imu_" parent="$(arg prefix)base_link">
+    <origin xyz="0.0 0.0 0.0" rpy="0 0 0"/>
+  </xacro:sensor_imu>
+  <!-- Gazebo ros control plugins -->
+  <xacro:arg name="config_controllers" default="$(find robot_description)/config/summit_xl_base.yaml"/>
+  <xacro:arg name="update_rate" default="100"/>
+  <xacro:include filename="$(find robot_description)/urdf/ros2_control.urdf.xacro"/>
+  <xacro:ros2_control/>
 </robot>
