Commit message: Support for Gazebo Harmonic

File: urdf/bases/summit_xl_base.urdf.xacro (robot description, xacro)
@@ -41,7 +41,7 @@
 		   </geometry>
 		   </xacro:unless>
-		   <material name="darkgrey">
+<!-- 		   <material name="darkgrey">
 			 <color rgba="0.1 0.1 0.1 1"/>
-		   </material>
+		   </material> -->
 		</visual>
 		<collision>

File: urdf/wheels/rubber_wheel/rubber_wheel.urdf.xacro (robot description, xacro)
@@ -7,16 +7,16 @@
               izz="${m*(3*r*r+h*h)/12}" />
   </xacro:macro>
-  <xacro:macro name="rubber_wheel" params="prefix parent *origin *axis reflect hq rubber_wheel_radius:=0.11 rubber_wheel_width:=0.15 rubber_wheel_mass:=6.5
+  <xacro:macro name="rubber_wheel" params="prefix parent *origin reflect hq rubber_wheel_radius:=0.11 rubber_wheel_width:=0.15 rubber_wheel_mass:=6.5
                                           mesh_file:=robot_description/meshes/wheels/rubber_wheel/rubber_wheel_right">
 <!--WHEEL TIRE -->
-    <joint name="${prefix}_wheel_joint" type="continuous">
+    <joint name="${prefix}wheel_joint" type="continuous">
       <parent link="${parent}"/>
-      <child link="${prefix}_wheel"/>
+      <child link="${prefix}wheel_link"/>
       <xacro:insert_block name="origin" />
-      <xacro:insert_block name="axis" />
+      <axis xyz="0 1 0" />
       <limit effort="100" velocity="100"/>
-      <joint_properties damping="0.0" friction="0.0"/>
+			<joint_properties damping="0.0" friction="0.0"/>
     </joint>
-    <link name="${prefix}_wheel">
+    <link name="${prefix}wheel_link">
       <visual>
         <!-- HIGH RESOLUTION WHEELS -->
@@ -58,18 +58,12 @@
     </link>
     <!-- Transmission is important to link the joints and the controller (see summit_xl_control/config/summit_xl_control.yaml)-->
-    <transmission name="${prefix}_wheel_joint_trans">
-      <type>transmission_interface/SimpleTransmission</type>
-      <joint name="${prefix}_wheel_joint">
-        <hardwareInterface>hardware_interface/VelocityJointInterface</hardwareInterface>
-      </joint>
-      <actuator name="${prefix}_wheel_joint_motor">
+    <transmission name="${prefix}wheel_joint_trans">
+      <plugin>transmission_interface/SimpleTransmission</plugin>
+      <actuator name="${prefix}wheel_joint_motor" role="actuator1"/>
+      <joint name="${prefix}wheel_joint" role="joint1">
         <mechanicalReduction>1</mechanicalReduction>
         <motorTorqueConstant>20</motorTorqueConstant>
-      </actuator>
+      </joint>
      </transmission>
-    <gazebo reference="${prefix}_wheel">
-			<material>Gazebo/Black</material>
-			<turnGravityOff>false</turnGravityOff>
-		</gazebo>
   </xacro:macro>
 </robot>

Commit message: fix: removed double underscore for gps__link

File: robots/summit_xl_std.urdf.xacro (robot description, xacro)
@@ -69,9 +69,9 @@
       <origin xyz="0.324 0.012 0.172" rpy="0 0 0"/>
   </xacro:sensor_stereolabs_zed2>
-  <xacro:structure_mastil_gps prefix="$(arg prefix)gps_" parent="$(arg prefix)base_link">
+  <xacro:structure_mastil_gps prefix="$(arg prefix)gps_base" parent="$(arg prefix)base_link">
     <origin xyz="-0.24 0.095 0.25" rpy="0 0 0"/>
   </xacro:structure_mastil_gps>
-  <xacro:sensor_gps  node_namespace="$(arg robot_ns)" frame_prefix="$(arg prefix)gps_" parent="$(arg prefix)base_link" simulation="true">
-    <origin xyz="-0.24 0.095 0.625" rpy="0 0 0"/>
+  <xacro:sensor_gps  node_namespace="$(arg robot_ns)" frame_prefix="$(arg prefix)gps_" parent="$(arg prefix)gps_base_link" simulation="true">
+    <origin xyz="0 0 0.375" rpy="0 0 0"/>
   </xacro:sensor_gps>
   <xacro:sensor_imu ns="$(arg robot_ns)" prefix="$(arg prefix)imu" parent="$(arg prefix)base_link">

File: urdf/structures/sensor_support/structure_gps.urdf.xacro (robot description, xacro)
@@ -2,5 +2,5 @@
 <robot name="structure" xmlns:xacro="http://wiki.ros.org/xacro">
   <xacro:macro name="structure_mastil_gps" params="prefix parent *origin">
-	  <joint name="${prefix}_joint" type="fixed">
+	  <joint name="${prefix}_mast_joint" type="fixed">
 	    <axis xyz="0 1 0"/>
 	    <xacro:insert_block name="origin"/>
